Commit message: sinking ship, saving data, bye ubuntu

File: isaac_flapper/Flapper-Env/resources/spm-asm-v6-2/urdf/spm-asm-v6-2.urdf (robot description, URDF)
Before this commit: robot spm-asm-v6-2, 5 links, 4 joints
Links:
- link IMU: geometry collision mesh filename=/home/afarah/Documents/UML/willis/rluff/isaac_flapper/Flapp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; visual mesh filename=/home/afarah/Documents/UML/willis/rluff/isaac_flapper/Flapp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
- link body: geometry collision mesh filename=/home/afarah/Documents/UML/willis/rluff/isaac_flapper/Flapp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; visual mesh filename=/home/afarah/Documents/UML/willis/rluff/isaac_flapper/Flapp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
- link egg: geometry collision mesh filename=/home/afarah/Documents/UML/willis/rluff/isaac_flapper/Flapp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; visual mesh filename=/home/afarah/Documents/UML/willis/rluff/isaac_flapper/Flapp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
- link left: geometry collision mesh filename=/home/afarah/Documents/UML/willis/rluff/isaac_flapper/Flapp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; visual mesh filename=/home/afarah/Documents/UML/willis/rluff/isaac_flapper/Flapp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
- link right: geometry collision mesh filename=/home/afarah/Documents/UML/willis/rluff/isaac_flapper/Flapp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; visual mesh filename=/home/afarah/Documents/UML/willis/rluff/isaac_flapper/Flapp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
